File: Schede/Girello2021/IO-Nano_r01/IO-Nano.kicad_pcb (KiCad board)
At the start: 2 copper layers, 10 parts, among them Q1 IRF540N, U1 L7805

Commit message: nanor1 - windows
Parts:
- added D2: LED, LED_THT:LED_D3.0mm, F.Cu at (120.7, -297.2)
- added D3: LED, LED_THT:LED_D3.0mm, F.Cu at (93.3, -295.7)
- added D4: LED, LED_THT:LED_D3.0mm, F.Cu at (118.1, -313.8)
- added D5: LED, LED_THT:LED_D3.0mm, F.Cu at (118.1, -308.3)
- added D6: LED, LED_THT:LED_D3.0mm, F.Cu at (118.1, -302.7)
- added OUT1: Screw_Terminal_01x02, TerminalBlock_Phoenix:TerminalBlock_Phoenix_MKDS-1,5-2-5.08_1x02_P5.08mm_Horizontal, F.Cu at (70.7, -306.0)
- added OUT2: Screw_Terminal_01x02, TerminalBlock_Phoenix:TerminalBlock_Phoenix_MKDS-1,5-2-5.08_1x02_P5.08mm_Horizontal, F.Cu at (85.4, -310.4)
- added OUT3: Screw_Terminal_01x02, TerminalBlock:TerminalBlock_bornier-2_P5.08mm, F.Cu at (97.3, -312.1)
- added OUT4: Screw_Terminal_01x02, TerminalBlock_Phoenix:TerminalBlock_Phoenix_MKDS-1,5-2-5.08_1x02_P5.08mm_Horizontal, F.Cu at (82.9, -298.5)
- added OUT5: Screw_Terminal_01x02, TerminalBlock:TerminalBlock_bornier-2_P5.08mm, F.Cu at (97.3, -303.0)
- added OUT6: Screw_Terminal_01x02, TerminalBlock_Phoenix:TerminalBlock_Phoenix_MKDS-1,5-2-5.08_1x02_P5.08mm_Horizontal, F.Cu at (70.7, -294.2)
- added Q2: IRF540N, Package_TO_SOT_THT:TO-220-3_Vertical, F.Cu at (82.6, -289.0)
- added RN1: R_220, Resistor_THT:R_Array_SIP5, F.Cu at (69.4, -314.4)
- added RV6: R_POT_1k, Potentiometer_THT:Potentiometer_Vishay_T73YP_Vertical, F.Cu at (45.7, -301.0)
- added RV7: R_POT_1k, Potentiometer_THT:Potentiometer_Vishay_T73YP_Vertical, F.Cu at (38.1, -260.4)
- added Rgnd1: R47, Resistor_THT:R_Axial_DIN0204_L3.6mm_D1.6mm_P7.62mm_Horizontal, F.Cu at (68.6, -287.0)
- added Ue1: PS2501, Package_DIP:DIP-4_W7.62mm, F.Cu at (107.2, -301.1)
- added Ue2: PS2501, Package_DIP:DIP-4_W7.62mm, F.Cu at (107.2, -307.8)
- added Ue3: PS2501, Package_DIP:DIP-4_W7.62mm, F.Cu at (92.5, -290.8)
- added Ue4: PS2501, Package_DIP:DIP-4_W7.62mm, F.Cu at (107.2, -314.5)
- moved Ro1 8.43 mm to (45.7, -287.0)
- moved c1 3.81 mm to (33.0, -308.6)
Connections:
- 24v-GND1 pad 2: GND -> Net-(24v-GND1-Pad2)
- 5v-GND1 pad 2: GND -> Net-(24v-GND1-Pad2)
- C2 pad 2: GND -> Net-(24v-GND1-Pad2)
- D1 pad 2: Net-(A1-Pad9) -> Net-(D1-Pad2)
- Q1 pad 1: Net-(A1-Pad9) -> Net-(D1-Pad2)
- Q1 pad 2: +24V -> Net-(OUT1-Pad1)
- U1 pad 2: GND -> Net-(24v-GND1-Pad2)
- c1 pad 1: GND -> Net-(24v-GND1-Pad2)
Other:
- net class Default: trace_width 0.5 -> 0.25
- net class Power added: clearance 0.2, trace_width 0.5, via_dia 0.8, via_drill 0.4
