File: Schede/Girello2021/IO-Nano_r01/IO-Nano.sch (KiCad schematic (older format))
At the start: 26 parts, among them Q1 IRF540N, Q2 IRF540N, U1 L7805

Commit message: nanor1 - windows
Parts:
- removed Ro1, Ro2, Ro3, Ro4, Ruo3, Ruo4: R220, Resistor_THT:R_Axial_DIN0204_L3.6mm_D1.6mm_P7.62mm_Horizontal, symbol Device:R
- added D5, D6: LED, LED_THT:LED_D3.0mm, symbol Device:LED
- added OUT5: Screw_Terminal_01x02, TerminalBlock:TerminalBlock_bornier-2_P5.08mm, symbol Connector:Screw_Terminal_01x02
- added OUT6: Screw_Terminal_01x02, TerminalBlock_Phoenix:TerminalBlock_Phoenix_MKDS-1,5-2-5.08_1x02_P5.08mm_Horizontal, symbol Connector:Screw_Terminal_01x02
- added RN1: R_220, Resistor_THT:R_Array_SIP5, symbol Device:R_Network04
- added RV6, RV7: R_POT_1k, Potentiometer_THT:Potentiometer_Vishay_T73YP_Vertical, symbol Device:R_POT_TRIM
- added Ue1, Ue2: PS2501, Package_DIP:DIP-4_W7.62mm, symbol Isolator:PC817
- renumbered Uo4 to Ue3, Uo3 to Ue4
Connections:
- net labels added: 10-13_Eth
- wire segments 91 -> 83
Other:
- moved on the sheet: D1, OUT1, OUT2, OUT3, OUT4, Q1, Q2, Rgnd1, Ue3, Ue4

Commit message: -
Parts:
- added U11: DOIT-ESP32-30PIN, ESP8266:ESP-12, symbol ESP32-DOIT:DOIT-ESP32-30PIN
Connections:
- wire segments 83 -> 87
Changed lines of the file:
@@
 $EndComp
-Wire Wire Line
-	5550 5050 5550 5150
 Wire Wire Line
 	5550 5150 6200 5150
@@
 Wire Wire Line
 	7100 4000 6950 4000
+Wire Wire Line
+	3750 2350 3750 2150
+Wire Wire Line
+	3750 2150 5550 2150
+Connection ~ 5550 2150
+$Comp
+L ESP32-DOIT:DOIT-ESP32-30PIN U11
+U 1 1 602EEC5A
+P 1950 5250
+F 0 "U11" H 1925 5815 50  0000 C CNN
+F 1 "DOIT-ESP32-30PIN" H 1925 5724 50  0000 C CNN
+F 2 "ESP8266:ESP-12" H 1900 5700 50  0001 C CNN
+F 3 "" H 1900 5700 50  0001 C CNN
+	1    1950 5250
+	1    0    0    -1
+$EndComp
+Wire Wire Line
+	2550 6250 5550 6250
+Wire Wire Line
+	5550 5050 5550 5150
+Connection ~ 5550 5150
+Wire Wire Line
+	5550 5150 5550 6250
 $EndSCHEMATC
