File: Schede/IO-ESP32-30-Relay/IO-ESP32-30-Relay.kicad_pcb (KiCad board)
At the start: 2 copper layers, 43.2 x 72.4 mm, 18 parts, among them J1 pinHeaderR, J2 Screw_Terminal_01x08, U1 DOIT-ESP32-30PIN

Commit message: esp32
Parts:
- removed 3v3-GND: Screw_Terminal_01x02, TerminalBlock_Phoenix:TerminalBlock_Phoenix_MKDS-1,5-2-5.08_1x02_P5.08mm_Horizontal
- added 3v3: Screw_Terminal_01x02, TerminalBlock_Phoenix:TerminalBlock_Phoenix_MKDS-1,5-2-5.08_1x02_P5.08mm_Horizontal, F.Cu at (101.6, 146.1)
- J1: value pinHeaderR -> PinHeader_4x2Relay
- renumbered 5V-GND to 5V1
Connections:
- 5V1 pad 2: Net-(3v3-GND1-Pad2) -> GND
- J1 pad 6: Net-(J1-Pad6) -> GND
- J1 pad 7: Net-(J1-Pad6) -> GND
- RN1 pad 1: Net-(3v3-GND1-Pad2) -> GND
- RN2 pad 1: Net-(3v3-GND1-Pad2) -> GND
- U1 pad 14: Net-(3v3-GND1-Pad2) -> GND
- U1 pad 17: Net-(J1-Pad6) -> GND
Routing:
- net GND: track 0.00 -> 169.3 mm
- net Net-(3v3-GND1-Pad2): track 126.1 -> 0.00 mm
- net Net-(J1-Pad6): track 43.1 -> 0.00 mm
Other:
- net class Power added: clearance 0.4, trace_width 0.5, via_dia 0.8, via_drill 0.4
